Commit message: added vacuum gripper to gazebo

File: src/enme480_description/urdf/enme480_ur3e_macro.xacro (robot description, xacro)
@@ -89,27 +89,31 @@
       <origin rpy="0 0 0" xyz="0 ${-mount_width/2} ${stand_height}"/>
     </joint>
-<!-- !!!end effector definition!!! -->
-    <link name="${tf_prefix}ee_mount_link">
-      <visual>
-        <geometry>
-          <mesh filename="file://$(find enme480_description)/meshes/ee_mount/ee_mount.stl"/>
-        </geometry>
-        <material name="VeryDarkGray">
-          <color rgba="0.3 0.3 0.3 1.0"/>
-        </material>
-        <origin rpy="0.0 ${pi} 0.0" xyz="0.0 0.0 0.008"/>
-      </visual>
-      <collision>
-        <geometry>
-          <box size="0.02 0.04675 0.0435"/>
-        </geometry>
+    <gazebo reference="${tf_prefix}wood_top">
+      <collision>
         <surface>
           <friction>
             <ode>
-              <mu>10000</mu>
-              <mu2>10000</mu2>
+              <mu>0.3</mu>
+              <mu2>0.3</mu2>
             </ode>
           </friction>
         </surface>
+      </collision>
+    </gazebo>
+<!-- !!!end effector definition!!! -->
+    <link name="${tf_prefix}ee_mount_link">
+      <visual>
+        <geometry>
+          <mesh filename="file://$(find enme480_description)/meshes/ee_mount/ee_mount.stl"/>
+        </geometry>
+        <material name="VeryDarkGray">
+          <color rgba="0.3 0.3 0.3 1.0"/>
+        </material>
+        <origin rpy="0.0 ${pi} 0.0" xyz="0.0 0.0 0.008"/>
+      </visual>
+      <collision>
+        <geometry>
+          <box size="0.02 0.04675 0.0435"/>
+        </geometry>
         <origin rpy="0.0 0.0 0.0" xyz="0.0 ${-(0.0315+0.04675)/2} ${0.0435/2}"/>
       </collision>
@@ -125,4 +129,7 @@
       <origin rpy="0.0 ${pi/2.0} 0.0" xyz="0 0.0 0.0"/>
     </joint>
+    <gazebo reference="${tf_prefix}ee_fixed_joint">
+      <preserveFixedJoint>true</preserveFixedJoint>
+    </gazebo>
     <gazebo reference="${tf_prefix}ee_mount_link">
       <material>Gazebo/Grey</material>
@@ -143,12 +150,4 @@
           <cylinder radius="${0.0175/2}" length="0.0145"/>
         </geometry>
-        <surface>
-          <friction>
-            <ode>
-              <mu>10000</mu>
-              <mu2>10000</mu2>
-            </ode>
-          </friction>
-        </surface>
         <origin rpy="0.0 0.0 0.0" xyz="0.0 0.0 ${-0.0145/2}"/>
       </collision>
@@ -167,6 +166,69 @@
       <dynamics damping="0.0" friction="10"/> -->
     </joint>
+    <gazebo reference="${tf_prefix}gripper_joint">
+      <preserveFixedJoint>true</preserveFixedJoint>
+    </gazebo>
     <gazebo reference="${tf_prefix}vac_gripper">
       <material>Gazebo/Black</material>
+    </gazebo>
+    <!-- Suction sensor vac_gripper-->
+    <link name="suction_link">
+      <gravity>0</gravity>
+      <visual>
+        <geometry>
+          <cylinder radius="0.009" length="0.002"/>
+        </geometry>
+        <material name="suction_red">
+          <color rgba="1.0 0.0 0.0 1.0"/>
+        </material>
+        <origin rpy="0.0 0.0 0.0" xyz="0.0 0.0 0.0"/>
+      </visual>
+      <collision>
+        <geometry>
+          <cylinder radius="0.009" length="0.002"/>
+        </geometry>
+        <origin rpy="0.0 0.0 0.0" xyz="0.0 0.0 0.0"/>
+      </collision>
+      <inertial>
+        <origin rpy="0 0 0" xyz="0.0 0.0 0.0"/>
+        <mass value="0.0001"/>
+        <inertia ixx="1e-08" ixy="0" ixz="0" iyy="1e-08" iyz="0" izz="1e-08"/>
+      </inertial>
+    </link>
+    <joint name="suction_joint" type="fixed">
+      <parent link="vac_gripper" />
+      <child link="suction_link" />
+      <origin rpy="0.0 0.0 0.0" xyz="0.0 0.0 0.0" />
+    </joint>
+    <gazebo reference="suction_joint">
+      <preserveFixedJoint>true</preserveFixedJoint>
+    </gazebo>
+    <gazebo reference="suction_link">
+      <material>Gazebo/Red</material>
+      <collision>
+        <surface>
+          <friction>
+            <ode>
+              <mu>10</mu>
+              <mu2>10</mu2>
+            </ode>
+          </friction>
+        </surface>
+      </collision>
+      <sensor name='contact_sensor_0' type='contact'>
+        <update_rate>10</update_rate>
+        <always_on>1</always_on>
+        <contact>
+          <collision>suction_link_collision</collision>
+          <topic>/gripper/contact_sensor_0</topic>
+        </contact>
+      </sensor>
+    </gazebo>
+    <gazebo>
+      <plugin filename="libVacuumGripper.so" name="mrc_gazebo_plugins::VacuumGripperPlugin">
+        <parent_link>suction_link</parent_link>
+        <contact_sensor_topic_prefix>/gripper</contact_sensor_topic_prefix>
+        <command_topic>/gripper/vac_on</command_topic>
+      </plugin>
     </gazebo>
     <!--This will create the specific robot-->
